File: AliceBoardPCB/AliceBoardPCB.kicad_pcb (KiCad board)
At the start: 2 copper layers, 146 parts, among them SW1 SW_PUSH, U1 ATmega32U4-AU, U2 PRTR5V0U2X, Y1 16Mhz

Commit message: PCB Update
more pcb updates
Parts:
- moved D6 7.30 mm to (95.2, 92.1), turned to 90 degrees
- moved D3 7.06 mm to (77.4, 130.5), turned to 90 degrees
- moved D45 7.03 mm to (281.7, 129.0), turned to 98 degrees
- moved D4 7.00 mm to (79.1, 149.5), turned to 90 degrees
- moved D5 7.00 mm to (69.6, 168.4), turned to 90 degrees
- moved D19 6.99 mm to (154.0, 97.6), turned to 82 degrees
- moved D40 6.98 mm to (262.8, 131.7), turned to 98 degrees
- moved D42 6.97 mm to (275.4, 168.5), turned to 98 degrees
- moved D34 6.96 mm to (236.4, 116.2), turned to 98 degrees
- moved D39 6.94 mm to (255.3, 113.6), turned to 98 degrees
- moved D46 6.93 mm to (274.9, 149.3), turned to 98 degrees
- moved D9 6.93 mm to (110.3, 149.5), turned to 90 degrees
- moved D32 6.92 mm to (218.3, 157.3), turned to 98 degrees
- moved D48 6.92 mm to (294.5, 110.9), turned to 90 degrees
- moved D44 6.91 mm to (274.1, 111.0), turned to 98 degrees
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Routing:
- net ROW3: track 0.00 -> 266.9 mm
- net ROW0: track 0.00 -> 252.4 mm
- net ROW1: track 0.00 -> 250.1 mm
- net ROW4: track 0.00 -> 249.6 mm
- net ROW2: track 0.00 -> 240.3 mm
- net COL12: track 0.00 -> 96.9 mm
- net COL3: track 0.00 -> 87.6 mm
- net COL9: track 0.00 -> 87.1 mm
- net COL7: track 0.00 -> 87.1 mm
- net COL2: track 0.00 -> 86.8 mm
- net COL13: track 0.00 -> 86.1 mm
- net COL5: track 0.00 -> 85.0 mm
- net COL0: track 0.00 -> 82.3 mm
- net COL10: track 0.00 -> 68.6 mm
- net COL11: track 0.00 -> 68.4 mm
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
Commit message: First Draft!
I finished my first draft for the PCB. Im gonna work on making it look better and stuff but other than that its most likely functional and yea! Super excited to where this is going.
Parts:
- C1, C2, C3, C4, C5, C6, C7, C8, D1, D10, D11, D12, D13, D14, D15, D16, D17, D18, D19, D2, D20, D21, D22, D23, D24, D25, D26, D27, D28, D29, D3, D30, D31, D32, D33, D34, D35, D36, D37, D38, D39, D4, D40, D41, D42, D43, D44, D45, D46, D47, D48, D49, D5, D50, D51, D52, D53, D54, D55, D56, D57, D58, D59, D6, D60, D61, D62, D63, D7, D8, D9, F1, R1, R2, R3, R4, R5, R6, SW1, U1, U2, USB1, Y1: moved to B.Cu
- moved C2 103.8 mm to (199.2, 149.3), turned to 270 degrees
- moved U1 99.9 mm to (195.3, 137.3), turned to 180 degrees
- moved Y1 99.1 mm to (195.2, 149.3)
- moved C1 98.4 mm to (191.2, 149.3), turned to 270 degrees
- moved C3 95.1 mm to (203.8, 136.1), turned to 90 degrees
- moved R1 94.9 mm to (204.1, 99.5), turned to 90 degrees
- moved R2 94.2 mm to (206.9, 99.5), turned to 270 degrees
- moved C6 92.0 mm to (205.8, 137.1), turned to 90 degrees
- moved C8 89.2 mm to (205.8, 133.3), turned to 270 degrees
- moved C4 88.7 mm to (186.5, 135.8), turned to 90 degrees
- moved C7 87.3 mm to (204.7, 128.7), turned to 180 degrees
- moved F1 85.5 mm to (201.4, 96.8), turned to 270 degrees
- moved SW1 85.2 mm to (195.8, 122.6)
- moved R4 84.6 mm to (208.2, 92.9), turned to 90 degrees
- moved C5 82.8 mm to (186.2, 140.8), turned to 270 degrees
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Connections:
- U1 pad 10: Net-(U1-Pad10) -> COL8
- U1 pad 11: Net-(U1-Pad11) -> COL7
- U1 pad 12: Net-(U1-Pad12) -> COL6
- U1 pad 15: +5V -> GND
- U1 pad 18: Net-(U1-Pad18) -> ROW4
- U1 pad 19: Net-(U1-Pad19) -> ROW3
- U1 pad 20: Net-(U1-Pad20) -> ROW2
- U1 pad 21: Net-(U1-Pad21) -> ROW1
- U1 pad 22: Net-(U1-Pad22) -> ROW0
- U1 pad 23: +5V -> GND
- U1 pad 25: Net-(U1-Pad25) -> COL3
- U1 pad 26: Net-(U1-Pad26) -> COL2
- U1 pad 27: Net-(U1-Pad27) -> COL4
- U1 pad 28: Net-(U1-Pad28) -> COL5
- U1 pad 29: Net-(U1-Pad29) -> COL1
- U1 pad 30: Net-(U1-Pad30) -> COL0
- U1 pad 35: +5V -> GND
- U1 pad 39: Net-(U1-Pad39) -> COL13
- U1 pad 40: Net-(U1-Pad40) -> COL12
- U1 pad 41: Net-(U1-Pad41) -> COL11
- U1 pad 43: +5V -> GND
- U1 pad 5: +5V -> GND
- U1 pad 8: Net-(U1-Pad8) -> COL10
- U1 pad 9: Net-(U1-Pad9) -> COL9
Routing:
- net COL13: track 86.1 -> 272.0 mm, vias 0 -> 2
- net GND: track 0.00 -> 163.4 mm, vias 0 -> 3
- net COL12: track 96.9 -> 254.8 mm, vias 0 -> 2
- net COL0: track 82.3 -> 222.9 mm, vias 0 -> 2
- net COL11: track 68.4 -> 200.3 mm, vias 0 -> 2
- net +5V: track 0.00 -> 116.2 mm, vias 0 -> 5
- net COL1: track 63.8 -> 172.0 mm, vias 0 -> 2
- net ROW4: track 249.6 -> 349.1 mm, vias 0 -> 4
- net COL10: track 68.6 -> 167.1 mm, vias 0 -> 2
- net COL2: track 86.8 -> 170.2 mm, vias 0 -> 2
- net ROW1: track 250.1 -> 332.6 mm, vias 0 -> 4
- net ROW0: track 252.4 -> 332.0 mm, vias 0 -> 4
- net COL9: track 87.1 -> 163.6 mm, vias 0 -> 2
- net COL3: track 87.6 -> 151.2 mm, vias 0 -> 2
- net ROW3: track 266.9 -> 330.1 mm, vias 0 -> 3
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- added copper zone on B.Cu, net GND
Other:
- board outline added: 317.1 x 108.4 mm

Commit message: Finished PCB
Less Gooooo
Parts:
- MX14: footprint MX_Only:MXOnly-1U-NoLED -> MX_Only:MXOnly-2U-NoLED
- MX15, MX28: footprint MX_Only:MXOnly-1U-NoLED -> MX_Only:MXOnly-1.5U-NoLED
- MX29, MX54: footprint MX_Only:MXOnly-1U-NoLED -> MX_Only:MXOnly-1.75U-NoLED
- MX41, MX42, MX58: footprint MX_Only:MXOnly-1U-NoLED -> MX_Only:MXOnly-2.25U-NoLED
- MX56, MX61, MX62, MX63: footprint MX_Only:MXOnly-1U-NoLED -> MX_Only:MXOnly-1.25U-NoLED
- MX60: footprint MX_Only:MXOnly-1U-NoLED -> MX_Only:MXOnly-2.75U-NoLED
- moved F1 3.01 mm to (204.4, 97.0)
- moved R1 3.01 mm to (207.1, 99.7)
- moved R3 3.01 mm to (206.0, 91.2)
- moved U2 3.01 mm to (208.5, 95.1)
- moved USB1 3.01 mm to (208.4, 79.9)
- moved R4 3.01 mm to (211.2, 93.1)
- moved R2 2.12 mm to (209.1, 99.7)
- moved C5 0.87 mm to (186.6, 141.6)
- moved D61 0.26 mm to (349.4, 92.2)
- moved MX14 0.26 mm to (341.1, 92.2)
- moved D56 0.23 mm to (320.8, 92.3)
- moved MX13 0.23 mm to (312.5, 92.2)
- moved C3 0.10 mm to (203.8, 136.0)
Connections:
- U1 pad 21: ROW1 -> COL5
- U1 pad 22: ROW0 -> COL4
- U1 pad 27: COL4 -> COL1
- U1 pad 28: COL5 -> COL0
- U1 pad 29: COL1 -> Net-(U1-Pad29)
- U1 pad 30: COL0 -> Net-(U1-Pad30)
- U1 pad 37: Net-(U1-Pad37) -> ROW0
- U1 pad 38: Net-(U1-Pad38) -> ROW1
- U1 pad 39: COL13 -> COL11
- U1 pad 41: COL11 -> COL13
Routing:
- net GND: track 163.4 -> 125.9 mm
- net +5V: track 116.2 -> 141.2 mm, vias 5 -> 8
- net ROW1: track 332.6 -> 314.5 mm, vias 4 -> 2
- net ROW0: track 332.0 -> 319.2 mm
- net COL5: track 114.0 -> 109.3 mm, vias 2 -> 0
- net COL4: track 111.7 -> 107.7 mm, vias 2 -> 0
- net ROW3: track 330.1 -> 327.2 mm
- net COL11: track 200.3 -> 202.7 mm
- net COL6: track 98.0 -> 96.5 mm, vias 2 -> 0
- net Net-(R2-Pad2): track 44.1 -> 45.4 mm
- net COL2: track 170.2 -> 171.4 mm, vias 2 -> 0
- net Net-(R5-Pad2): track 23.1 -> 24.2 mm
- net COL13: track 272.0 -> 271.0 mm
- net Net-(R1-Pad1): track 43.1 -> 43.9 mm
- net COL3: track 151.2 -> 151.8 mm, vias 2 -> 0
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Other:
- board size 317.1 x 108.4 mm -> 319.5 x 109.4 mm
- board text added: "Designed by AltaFour in Colorado"
